Commit message: feat: add camera_optical_link
Signed-off-by: Shin-kyoto <aquashin0202@gmail.com>

File: aichallenge/workspace/src/aichallenge_submit/racing_kart_sensor_kit_description/urdf/sensor_kit.xacro (robot description, xacro)
@@ -18,4 +18,31 @@
     <xacro:property name="calibration" value="${xacro.load_yaml('$(arg config_dir)/sensor_kit_calibration.yaml')}"/>
     <!-- over write calibration file for simulation -->
+    <xacro:if value="$(arg simulation)">
+      <xacro:property name="calibration" value="${xacro.load_yaml('$(arg config_dir)/awsim_sensor_kit_calibration.yaml')}"/>
+    </xacro:if>
+    <!-- camera -->
+    <joint name="camera_joint" type="fixed">
+      <origin rpy="${calibration['sensor_kit_base_link']['camera_link']['roll']} ${calibration['sensor_kit_base_link']['camera_link']['pitch']} ${calibration['sensor_kit_base_link']['camera_link']['yaw']}"
+              xyz="${calibration['sensor_kit_base_link']['camera_link']['x']} ${calibration['sensor_kit_base_link']['camera_link']['y']} ${calibration['sensor_kit_base_link']['camera_link']['z']}"/>
+      <parent link="sensor_kit_base_link"/>
+      <child link="camera_link"/>
+    </joint>
+    <link name="camera_link">
+      <visual>
+        <geometry>
+          <box size="0.1 0.1 0.1"/>
+        </geometry>
+        <material name="blue">
+          <color rgba="0 0 1 1"/>
+        </material>
+      </visual>
+    </link>
+    <joint name="camera_optical_joint" type="fixed">
+      <origin rpy="${-pi/2} 0 ${-pi/2}" xyz="0 0 0"/>
+      <parent link="camera_link"/>
+      <child link="camera_optical_link"/>
+    </joint>
+    <link name="camera_optical_link"/>
+    <xacro:property name="calibration" value="${xacro.load_yaml('$(arg config_dir)/sensor_kit_calibration.yaml')}"/>
     <xacro:if value="$(arg simulation)">
       <xacro:property name="calibration" value="${xacro.load_yaml('$(arg config_dir)/awsim_sensor_kit_calibration.yaml')}"/>
